File: Osciliscope PCB/ADC_Input.kicad_sch (KiCad schematic)
At the start: 30 parts, among them U4 OPA350UA_2K5, U5 OPA350UA_2K5

Commit message: Edited Schematic
Parts:
- added R19, R21: 10k, symbol Device:R
- added R20, R22: 30k, symbol Device:R
- C21, C31: footprint Diode_SMD:D_0805_2012Metric -> (none); Part NO. C14857 -> (none)
- C22, C24, C25, C26, C27: footprint Capacitor_SMD:C_0805_2012Metric -> (none); Part NO. C28233 -> (none)
- C23: footprint Capacitor_SMD:C_0805_2012Metric -> (none); Part NO. C377773 -> (none)
- R10, R11, R13, R15: footprint Resistor_SMD:R_0805_2012Metric -> (none); Part NO. C17514 -> (none)
- R12, R17, R18, R19, R20, R21, R22, R23, R25, R9: footprint Resistor_SMD:R_0805_2012Metric -> (none); Part NO. C26108 -> (none)
- R14, R16: footprint Resistor_SMD:R_0805_2012Metric -> (none); Part NO. C17408 -> (none)
- R7, R8: value 1M -> 10k; footprint Resistor_SMD:R_0805_2012Metric -> (none); Part NO. C17514 -> (none)
Connections:
- net GND: now also R19.1, R21.1
- net OPA1_OUT: now also R22.2; no longer U4.2 (-IN)
- net OPA2_OUT: now also R20.2; no longer U5.2 (-IN)
- new net: R21.2, R22.1, U4.2 (-IN)
- new net: R19.2, R20.1, U5.2 (-IN)

Commit message: Started main loop and added changes to screen function for allign
Parts:
- removed R20, R22: 30k, symbol Device:R
- added R29, R30: 30k, symbol Device:R
- renumbered R21 to R27, R19 to R28
Connections:
- net OPA1_OUT: now also R29.2
- net OPA2_OUT: now also R30.2
- net IN+1: now reaches R27.2, U4.2 (-IN)
- net IN+1: now also R29.1
- net IN+2: now reaches R28.2, U5.2 (-IN)
- net IN+2: now also R30.1
Changed lines of the file:
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@@
+		)
+	)
+	(label "IN+1"
+		(at 143.51 69.85 0)
+		(effects
+			(font
+				(size 1.27 1.27)
+			)
+			(justify left bottom)
 		)
 	)
@@
 	(label "OPA1_OUT"
 		(at 177.8 48.26 0)
+		(effects
+			(font
+				(size 1.27 1.27)
+			)
+			(justify left bottom)
+		)
+	)
+	(label "IN+2"
+		(at 144.78 118.11 0)
 		(effects
 			(font
@@
 		(dnp no)
 		(fields_autoplaced yes)
-		(property "Reference" "R?"
+		(property "Reference" "R27"
 			(at 139.7 73.6599 0)
 			(effects
@@
 			(project "Osciliscope PCB"
 				(path "/dbd44bf2-721f-49a6-94a9-d8437df40c50/df3a70e5-5419-4d97-af41-dbff22d05423"
-					(reference "R?")
+					(reference "R27")
 					(unit 1)
 				)
@@
 				(path "/dbd44bf2-721f-49a6-94a9-d8437df40c50/df3a70e5-5419-4d97-af41-dbff22d05423"
 					(reference "R25")
+					(unit 1)
+				)
+			)
+		)
+	)
+	(symbol
+		(lib_id "Device:R")
+		(at 161.29 118.11 90)
+		(mirror x)
+		(unit 1)
+		(exclude_from_sim no)
+		(in_bom yes)
+		(on_board yes)
+		(dnp no)
+		(property "Reference" "R30"
+			(at 161.29 124.46 90)
+			(effects
+				(font
+					(size 1.27 1.27)
+				)
+			)
+		)
+		(property "Value" "30k"
+			(at 161.29 121.92 90)
+			(effects
+				(font
+					(size 1.27 1.27)
+				)
+			)
+		)
+		(property "Footprint" ""
+			(at 161.29 116.332 90)
+			(effects
+				(font
+					(size 1.27 1.27)
+				)
+				(hide yes)
+			)
+		)
+		(property "Datasheet" ""
+			(at 161.29 118.11 0)
+			(effects
+				(font
+					(size 1.27 1.27)
+				)
+				(hide yes)
+			)
+		)
+		(property "Description" ""
+			(at 161.29 118.11 0)
+			(effects
+				(font
+					(size 1.27 1.27)
+				)
+				(hide yes)
+			)
+		)
+		(property "Part NO." ""
+			(at 161.29 118.11 0)
+			(effects
+				(font
+					(size 1.27 1.27)
+				)
+				(hide yes)
+			)
+		)
+		(pin "1"
+		)
+		(pin "2"
+		)
+		(instances
+			(project "Osciliscope PCB"
+				(path "/dbd44bf2-721f-49a6-94a9-d8437df40c50/df3a70e5-5419-4d97-af41-dbff22d05423"
+					(reference "R30")
 					(unit 1)
 				)
@@
 		(on_board yes)
 		(dnp no)
-		(property "Reference" "R?"
+		(property "Reference" "R29"
 			(at 158.75 76.2 90)
 			(effects
@@
 		)
 		(property "Part NO." ""
-			(at 158.75 69.85 90)
+			(at 158.75 69.85 0)
 			(effects
 				(font
@@
 		)
 		(instances
-			(project "ADC_Input"
-				(path "/2f23e878-87c8-4989-b421-e1f362801019"
-					(reference "R22")
-					(unit 1)
-				)
-			)
-			(project "Osciliscope PCB"
-				(path "/dbd44bf2-721f-49a6-94a9-d8437df40c50/df3a70e5-5419-4d97-af41-dbff22d05423"
-					(reference "R?")
+			(project "Osciliscope PCB"
+				(path "/dbd44bf2-721f-49a6-94a9-d8437df40c50/df3a70e5-5419-4d97-af41-dbff22d05423"
+					(reference "R29")
 					(unit 1)
 				)
@@
 		(dnp no)
 		(fields_autoplaced yes)
-		(property "Reference" "R?"
+		(property "Reference" "R28"
 			(at 140.97 121.9199 0)
 			(effects
@@
 			(project "Osciliscope PCB"
 				(path "/dbd44bf2-721f-49a6-94a9-d8437df40c50/df3a70e5-5419-4d97-af41-dbff22d05423"
-					(reference "R?")
+					(reference "R28")
 					(unit 1)
 				)
@@
 					(unit 1)
 				)
-			)
-		)
-	)
-	(symbol
-		(lib_id "Device:R")
-		(at 161.29 118.11 90)
-		(mirror x)
-		(unit 1)
-		(exclude_from_sim no)
-		(in_bom yes)
-		(on_board yes)
-		(dnp no)
-		(property "Reference" "R?"
-			(at 161.29 124.46 90)
-			(effects
-				(font
-					(size 1.27 1.27)
-				)
-			)
-		)
-		(property "Value" "30k"
-			(at 161.29 121.92 90)
-			(effects
-				(font
-					(size 1.27 1.27)
-				)
-			)
-		)
-		(property "Footprint" ""
-			(at 161.29 116.332 90)
-			(effects
-				(font
-					(size 1.27 1.27)
-				)
-				(hide yes)
-			)
-		)
-		(property "Datasheet" ""
-			(at 161.29 118.11 0)
-			(effects
-				(font
-					(size 1.27 1.27)
-				)
-				(hide yes)
-			)
-		)
-		(property "Description" ""
-			(at 161.29 118.11 0)
-			(effects
-				(font
-					(size 1.27 1.27)
-				)
-				(hide yes)
-			)
-		)
-		(pin "1"
-		)
-		(pin "2"
-		)
-		(instances
-			(project ""
-				(path "/2f23e878-87c8-4989-b421-e1f362801019"
-					(reference "R20")
-					(unit 1)
-				)
-			)
-			(project "Osciliscope PCB"
-				(path "/dbd44bf2-721f-49a6-94a9-d8437df40c50/df3a70e5-5419-4d97-af41-dbff22d05423"
-					(reference "R?")
-					(unit 1)
-				)

Commit message: Edited schematic
Parts:
- C21, C22, C24, C25, C26, C27, C31, R10, R11, R12, R13, R14, R15, R16, R17, R18, R19, R20, R21, R22, R23, R25, R27, R28, R29, R30, R7, R8, R9: footprint (none) -> Capacitor_SMD:C_0402_1005Metric
- C23: footprint (none) -> Capacitor_SMD:C_0603_1608Metric
Changed lines of the file:
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@@
 			)
 		)
-		(property "Footprint" ""
+		(property "Footprint" "Capacitor_SMD:C_0402_1005Metric"
 			(at 138.938 74.93 90)
 			(effects
@@
 			)
 		)
-		(property "Footprint" ""
+		(property "Footprint" "Capacitor_SMD:C_0402_1005Metric"
 			(at 129.2352 107.95 0)
 			(effects
@@
 			)
 		)
-		(property "Footprint" ""
+		(property "Footprint" "Capacitor_SMD:C_0402_1005Metric"
 			(at 130.048 41.91 90)
 			(effects
@@
 			)
 		)
-		(property "Footprint" ""
+		(property "Footprint" "Capacitor_SMD:C_0402_1005Metric"
 			(at 86.868 92.71 90)
 			(effects
@@
 			)
 		)
-		(property "Footprint" ""
+		(property "Footprint" "Capacitor_SMD:C_0402_1005Metric"
 			(at 64.008 43.18 90)
 			(effects
@@
 			)
 		)
-		(property "Footprint" ""
+		(property "Footprint" "Capacitor_SMD:C_0402_1005Metric"
 			(at 161.29 116.332 90)
 			(effects
@@
 			)
 		)
-		(property "Footprint" ""
+		(property "Footprint" "Capacitor_SMD:C_0402_1005Metric"
 			(at 28.9052 69.85 0)
 			(effects
@@
 			)
 		)
-		(property "Footprint" ""
+		(property "Footprint" "Capacitor_SMD:C_0402_1005Metric"
 			(at 158.75 68.072 90)
 			(effects
@@
 			)
 		)
-		(property "Footprint" ""
+		(property "Footprint" "Capacitor_SMD:C_0402_1005Metric"
 			(at 104.648 92.71 90)
 			(effects
@@
 			)
 		)
-		(property "Footprint" ""
+		(property "Footprint" "Capacitor_SMD:C_0402_1005Metric"
 			(at 39.878 78.74 90)
 			(effects
@@
 			)
 		)
-		(property "Footprint" ""
+		(property "Footprint" "Capacitor_SMD:C_0402_1005Metric"
 			(at 140.208 123.19 90)
 			(effects
@@
 			)
 		)
-		(property "Footprint" ""
+		(property "Footprint" "Capacitor_SMD:C_0402_1005Metric"
 			(at 72.898 43.18 90)
 			(effects
@@
 			)
 		)
-		(property "Footprint" ""
+		(property "Footprint" "Capacitor_SMD:C_0402_1005Metric"
 			(at 193.04 50.038 90)
 			(effects
@@
 			)
 		)
-		(property "Footprint" ""
+		(property "Footprint" "Capacitor_SMD:C_0402_1005Metric"
 			(at 109.728 54.61 90)
 			(effects
@@
 			)
 		)
-		(property "Footprint" ""
+		(property "Footprint" "Capacitor_SMD:C_0402_1005Metric"
 			(at 181.9148 88.9 0)
 			(effects
@@
 			)
 		)
-		(property "Footprint" ""
+		(property "Footprint" "Capacitor_SMD:C_0603_1608Metric"
 			(at 47.9552 82.55 0)
 			(effects
@@
 			)
 		)
-		(property "Footprint" ""
+		(property "Footprint" "Capacitor_SMD:C_0402_1005Metric"
 			(at 90.678 43.18 90)
 			(effects
@@
 			)
 		)
-		(property "Footprint" ""
+		(property "Footprint" "Capacitor_SMD:C_0402_1005Metric"
 			(at 81.788 43.18 90)
 			(effects
@@
 			)
 		)
-		(property "Footprint" ""
+		(property "Footprint" "Capacitor_SMD:C_0402_1005Metric"
 			(at 220.6752 105.41 0)
 			(effects
@@
 			)
 		)
-		(property "Footprint" ""
+		(property "Footprint" "Capacitor_SMD:C_0402_1005Metric"
 			(at 95.758 92.71 90)
 			(effects
@@
 			)
 		)
-		(property "Footprint" ""
+		(property "Footprint" "Capacitor_SMD:C_0402_1005Metric"
 			(at 69.088 92.71 90)
 			(effects
@@
 			)
 		)
-		(property "Footprint" ""
+		(property "Footprint" "Capacitor_SMD:C_0402_1005Metric"
 			(at 99.568 43.18 90)
 			(effects
@@
 			)
 		)
-		(property "Footprint" ""
+		(property "Footprint" "Capacitor_SMD:C_0402_1005Metric"
 			(at 39.878 66.04 90)
 			(effects
@@
 			)
 		)
-		(property "Footprint" ""
+		(property "Footprint" "Capacitor_SMD:C_0402_1005Metric"
 			(at 110.998 104.14 90)
 			(effects
@@
 			)
 		)
-		(property "Footprint" ""
+		(property "Footprint" "Capacitor_SMD:C_0402_1005Metric"
 			(at 193.04 99.568 90)
 			(effects
@@
 			)
 		)
-		(property "Footprint" ""
+		(property "Footprint" "Capacitor_SMD:C_0402_1005Metric"
 			(at 181.9148 39.37 0)
 			(effects
@@
 			)
 		)
-		(property "Footprint" ""
+		(property "Footprint" "Capacitor_SMD:C_0402_1005Metric"
 			(at 129.2352 58.42 0)
 			(effects
@@
 			)
 		)
-		(property "Footprint" ""
+		(property "Footprint" "Capacitor_SMD:C_0402_1005Metric"
 			(at 130.048 91.44 90)
 			(effects
@@
 			)
 		)
-		(property "Footprint" ""
+		(property "Footprint" "Capacitor_SMD:C_0402_1005Metric"
 			(at 77.978 92.71 90)
 			(effects
@@
 			)
 		)
-		(property "Footprint" ""
+		(property "Footprint" "Capacitor_SMD:C_0402_1005Metric"
 			(at 220.6752 55.88 0)
 			(effects
