File: Osciliscope PCB/Osciliscope PCB.kicad_pcb (KiCad board)
At the start: 2 copper layers, 74 x 53 mm, 79 parts, among them J1 TYPE-C_16PIN_2MD__073_, J10 Conn_01x02_Pin, J11 Conn_01x04_Pin, J2 Conn_01x04_Pin, J3 Conn_01x09_Pin, J4 Conn_01x05_Pin, J5 Conn_01x05_Pin, J6 Conn_01x04_Pin, J7 Conn_01x03_Pin, J8 Conn_01x02_Pin, J9 Conn_01x05_Pin, SW1 SW_SPDT, U1 STM32F405RGT6, U2 AMS1117-3.3, U3 USBLC6-2SC6, U4 OPA350UA_2K5, U5 OPA350UA_2K5, Y1 24MHz

Commit message: Edited Schematic
Parts:
- removed C1, C11, C14, C17, C18, C19, C20, C22, C24, C25, C26, C27, C3, C4, C5, C6, C7: 100n, Capacitor_SMD:C_0805_2012Metric
- removed C10, C9: 18pF, Capacitor_SMD:C_0805_2012Metric
- removed C12, C13, C2: 10u, Capacitor_SMD:C_0805_2012Metric
- removed C15, C16, C23: 2.2u, Capacitor_SMD:C_0805_2012Metric
- removed C21, C31: 47p, Diode_SMD:D_0805_2012Metric
- removed C8: 4.7u, Capacitor_SMD:C_0805_2012Metric
- removed D1, D5: BAT54SLT1G, Package_TO_SOT_SMD:SOT-23
- removed D2, D3: LED, LED_SMD:LED_0805_2012Metric
- removed FB1: 600R @ 100MHz, Capacitor_SMD:C_0805_2012Metric
- removed G***: LOGO, 02Footprints:Image_OSC
- removed J1: TYPE-C_16PIN_2MD__073_, 02Footprints:SHOUHAN_TYPE-C_16PIN_2MD__073_
- removed J10, J8: Conn_01x02_Pin, Connector_PinHeader_2.54mm:PinHeader_1x02_P2.54mm_Vertical
- removed J11, J2, J6: Conn_01x04_Pin, Connector_PinHeader_2.54mm:PinHeader_1x04_P2.54mm_Vertical
- removed J3: Conn_01x09_Pin, Connector_PinHeader_2.54mm:PinHeader_1x09_P2.54mm_Vertical
- removed J4, J5, J9: Conn_01x05_Pin, Connector_PinHeader_2.54mm:PinHeader_1x05_P2.54mm_Vertical
- removed J7: Conn_01x03_Pin, Connector_PinHeader_2.54mm:PinHeader_1x03_P2.54mm_Vertical
- removed R1, R3: 10k, Resistor_SMD:R_0805_2012Metric
- removed R10, R11, R13, R15, R7, R8: 1M, Resistor_SMD:R_0805_2012Metric
- removed R12, R17, R18, R19, R20, R21, R22, R23, R25, R9: 10M, Resistor_SMD:R_0805_2012Metric
- removed R14, R16: 100, Resistor_SMD:R_0805_2012Metric
- removed R2, R4, R5, R6: 5k1, Resistor_SMD:R_0805_2012Metric
- removed R24, R26: 330, Resistor_SMD:R_0805_2012Metric
- removed S1: KMR221GLFS, 02Footprints:SW_KMR221GLFS
- removed SW1: SW_SPDT, 02Footprints:SW-SMD_SSSS810701
- removed U1: STM32F405RGT6, Package_QFP:LQFP-64_10x10mm_P0.5mm
- removed U2: AMS1117-3.3, Package_TO_SOT_SMD:SOT-223-3_TabPin2
- removed U3: USBLC6-2SC6, Package_TO_SOT_SMD:SOT-23-6
- removed U4, U5: OPA350UA_2K5, 02Footprints:SOIC127P599X175-8N
- removed Y1: 24MHz, Crystal:Crystal_SMD_3225-4Pin_3.2x2.5mm
Routing:
- net +3.3V: track 332.3 -> 0.00 mm, vias 11 -> 0
- net /RESET: track 100.9 -> 0.00 mm
- net GND: track 100.6 -> 0.00 mm, vias 40 -> 0
- net /Encode_2: track 37.2 -> 0.00 mm, vias 5 -> 0
- net /LCD_MISO: track 36.5 -> 0.00 mm, vias 1 -> 0
- net /TIM5_2B: track 36.2 -> 0.00 mm
- net /TIM5_2A: track 36.0 -> 0.00 mm
- net /SWD_CLK: track 28.3 -> 0.00 mm
- net /CHL_Select: track 27.1 -> 0.00 mm
- net /USART1_TX: track 26.0 -> 0.00 mm
- net /SWD_IO: track 25.7 -> 0.00 mm
- net /USART1_RX: track 24.9 -> 0.00 mm
- net /LCD_SCK: track 24.7 -> 0.00 mm
- net +1V65: track 24.2 -> 0.00 mm, vias 3 -> 0
- net /Encode_1: track 23.6 -> 0.00 mm, vias 2 -> 0
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- removed copper zone on F.Cu, net +3.3V
- removed copper zone on B.Cu, net GND
Other:
- board outline removed
- board text removed: "1B/1A/SW/VCC/GND"
- board text removed: "2B/2A/SW/VCC/GND"
- board text removed: "CHL"
- board text removed: "DIY-Oscilloscope V1"
- board text removed: "IN1"
- board text removed: "IN2"
- board text removed: "LCD_SPI"
- board text removed: "Pause"
- board text removed: "Power"
- board text removed: "SD-SPI"
- board text removed: "SDA/SCL/AXIS"
- board text removed: "SWD"
- board text removed: "TX/RX"

Commit message: Finished PCB
Parts:
- added C1: 100n, Capacitor_SMD:C_0402_1005Metric, F.Cu at (147.5, 89.9)
- added C10: 18pF, Capacitor_SMD:C_0402_1005Metric, F.Cu at (141.4, 93.2)
- added C11: 100n, Capacitor_SMD:C_0402_1005Metric, F.Cu at (146.4, 95.4)
- added C12: 10u, Capacitor_SMD:C_0805_2012Metric, F.Cu at (171.5, 107.4)
- added C13: 10u, Capacitor_SMD:C_0805_2012Metric, F.Cu at (180.6, 120.2)
- added C14: 100n, Capacitor_SMD:C_0402_1005Metric, F.Cu at (169.4, 96.0)
- added C15: 2.2u, Capacitor_SMD:C_0603_1608Metric, F.Cu at (161.9, 91.0)
- added C16: 2.2u, Capacitor_SMD:C_0603_1608Metric, F.Cu at (157.5, 104.1)
- added C17: 100n, Capacitor_SMD:C_0402_1005Metric, F.Cu at (144.8, 91.6)
- added C18: 100n, Capacitor_SMD:C_0402_1005Metric, F.Cu at (146.4, 91.6)
- added C19: 100n, Capacitor_SMD:C_0402_1005Metric, F.Cu at (147.8, 100.8)
- added C2: 10u, Capacitor_SMD:C_0805_2012Metric, F.Cu at (149.2, 86.4)
- added C20: 100n, Capacitor_SMD:C_0402_1005Metric, F.Cu at (156.0, 87.6)
- added C21: 47p, Capacitor_SMD:C_0402_1005Metric, F.Cu at (150.9, 105.5)
- added C22: 100n, Capacitor_SMD:C_0402_1005Metric, F.Cu at (127.6, 104.6)
- added C23: 2.2u, Capacitor_SMD:C_0603_1608Metric, F.Cu at (130.4, 104.3)
- added C24: 100n, Capacitor_SMD:C_0402_1005Metric, F.Cu at (135.7, 112.4)
- added C25: 100n, Capacitor_SMD:C_0402_1005Metric, F.Cu at (144.6, 109.4)
- added C26: 100n, Capacitor_SMD:C_0402_1005Metric, F.Cu at (134.0, 105.8)
- added C27: 100n, Capacitor_SMD:C_0402_1005Metric, F.Cu at (142.9, 102.7)
- added C28: 100n, Capacitor_SMD:C_0402_1005Metric, F.Cu at (154.0, 85.6)
- added C3: 100n, Capacitor_SMD:C_0402_1005Metric, F.Cu at (150.7, 103.3)
- added C31: 47p, Capacitor_SMD:C_0402_1005Metric, F.Cu at (148.4, 102.4)
- added C4: 100n, Capacitor_SMD:C_0402_1005Metric, F.Cu at (150.1, 88.1)
- added C5: 100n, Capacitor_SMD:C_0402_1005Metric, F.Cu at (160.1, 90.4)
- added C6: 100n, Capacitor_SMD:C_0402_1005Metric, F.Cu at (159.3, 101.6)
- added C7: 100n, Capacitor_SMD:C_0402_1005Metric, F.Cu at (145.9, 96.9)
- added C8: 4.7u, Capacitor_SMD:C_0603_1608Metric, F.Cu at (143.2, 97.2)
- added C9: 18pF, Capacitor_SMD:C_0402_1005Metric, F.Cu at (141.8, 88.3)
- added D1: BAT54SLT1G, Package_TO_SOT_SMD:SOT-23, F.Cu at (146.7, 104.5)
- added D2: LED, Capacitor_SMD:C_0805_2012Metric, F.Cu at (172.0, 111.5)
- added D3: LED, Capacitor_SMD:C_0805_2012Metric, F.Cu at (172.0, 113.8)
- added D5: BAT54SLT1G, Package_TO_SOT_SMD:SOT-23, F.Cu at (150.2, 108.3)
- added FB1: 600R @ 100MHz, Capacitor_SMD:C_0805_2012Metric, F.Cu at (139.8, 96.9)
- added J1: TYPE-C_16PIN_2MD__073_, 02Footprints:SHOUHAN_TYPE-C_16PIN_2MD__073_, F.Cu at (189.2, 94.0)
- added J10: Conn_01x02_Pin, Connector_PinHeader_2.54mm:PinHeader_1x02_P2.54mm_Vertical, F.Cu at (175.0, 103.1)
- added J11: Conn_01x04_Pin, Connector_PinHeader_2.54mm:PinHeader_1x04_P2.54mm_Vertical, F.Cu at (127.7, 118.4)
- added J2: Conn_01x04_Pin, Connector_PinHeader_2.54mm:PinHeader_1x04_P2.54mm_Vertical, F.Cu at (167.4, 110.1)
- added J3: Conn_01x09_Pin, Connector_PinHeader_2.54mm:PinHeader_1x09_P2.54mm_Vertical, F.Cu at (147.2, 122.0)
- added J4: Conn_01x05_Pin, Connector_PinHeader_2.54mm:PinHeader_1x05_P2.54mm_Vertical, F.Cu at (169.4, 74.5)
- added J5: Conn_01x05_Pin, Connector_PinHeader_2.54mm:PinHeader_1x05_P2.54mm_Vertical, F.Cu at (129.1, 100.7)
- added J6: Conn_01x04_Pin, Connector_PinHeader_2.54mm:PinHeader_1x04_P2.54mm_Vertical, F.Cu at (140.9, 74.7)
- added J7: Conn_01x03_Pin, Connector_PinHeader_2.54mm:PinHeader_1x03_P2.54mm_Vertical, F.Cu at (154.3, 74.6)
- added J8: Conn_01x02_Pin, Connector_PinHeader_2.54mm:PinHeader_1x02_P2.54mm_Vertical, F.Cu at (179.5, 105.7)
- added J9: Conn_01x05_Pin, Connector_PinHeader_2.54mm:PinHeader_1x05_P2.54mm_Vertical, F.Cu at (179.5, 89.4)
- added R1: 10k, Capacitor_SMD:C_0402_1005Metric, F.Cu at (144.8, 95.0)
- added R10: 1M, Capacitor_SMD:C_0402_1005Metric, F.Cu at (132.6, 105.2)
- added R11: 1M, Capacitor_SMD:C_0402_1005Metric, F.Cu at (132.6, 107.2)
- added R12: 10M, Capacitor_SMD:C_0402_1005Metric, F.Cu at (130.3, 114.6)
- added R13: 1M, Capacitor_SMD:C_0402_1005Metric, F.Cu at (133.3, 112.9)
- added R14: 100, Capacitor_SMD:C_0402_1005Metric, F.Cu at (147.5, 107.6)
- added R15: 1M, Capacitor_SMD:C_0402_1005Metric, F.Cu at (133.1, 111.3)
- added R16: 100, Capacitor_SMD:C_0402_1005Metric, F.Cu at (146.0, 101.9)
- added R17: 10M, Capacitor_SMD:C_0402_1005Metric, F.Cu at (130.1, 110.5)
- added R18: 10M, Capacitor_SMD:C_0402_1005Metric, F.Cu at (130.6, 109.0)
- added R19: 10M, Capacitor_SMD:C_0402_1005Metric, F.Cu at (131.0, 107.4)
- added R2: 5k1, Capacitor_SMD:C_0402_1005Metric, F.Cu at (182.9, 95.3)
- added R20: 10M, Capacitor_SMD:C_0402_1005Metric, F.Cu at (131.5, 114.6)
- added R21: 10M, Capacitor_SMD:C_0402_1005Metric, F.Cu at (133.3, 115.2)
- added R22: 10M, Capacitor_SMD:C_0402_1005Metric, F.Cu at (135.2, 114.6)
- added R23: 10M, Capacitor_SMD:C_0402_1005Metric, F.Cu at (133.3, 114.0)
- added R24: 330, Capacitor_SMD:C_0603_1608Metric, F.Cu at (172.2, 109.2)
- added R25: 10M, Capacitor_SMD:C_0402_1005Metric, F.Cu at (127.6, 112.7)
- added R26: 330, Capacitor_SMD:C_0603_1608Metric, F.Cu at (172.2, 116.1)
- added R27: 10k, Capacitor_SMD:C_0402_1005Metric, F.Cu at (132.8, 103.2)
- added R28: 10k, Capacitor_SMD:C_0402_1005Metric, F.Cu at (134.4, 109.9)
- added R29: 30k, Capacitor_SMD:C_0402_1005Metric, F.Cu at (134.1, 103.2)
- added R3: 10k, Capacitor_SMD:C_0402_1005Metric, F.Cu at (150.1, 83.7)
- added R30: 30k, Capacitor_SMD:C_0402_1005Metric, F.Cu at (135.7, 109.9)
- added R4: 5k1, Capacitor_SMD:C_0402_1005Metric, F.Cu at (182.9, 92.3)
- added R5: 5k1, Capacitor_SMD:C_0402_1005Metric, F.Cu at (154.1, 77.1)
- added R6: 5k1, Capacitor_SMD:C_0402_1005Metric, F.Cu at (156.2, 77.1)
- added R7: 10k, Capacitor_SMD:C_0402_1005Metric, F.Cu at (127.6, 105.7)
- added R8: 10k, Capacitor_SMD:C_0402_1005Metric, F.Cu at (129.8, 105.7)
- added R9: 10M, Capacitor_SMD:C_0402_1005Metric, F.Cu at (128.9, 111.6)
- added S1: KMR221GLFS, 02Footprints:SW_KMR221GLFS, F.Cu at (135.6, 91.8)
- added SW1: SW_SPDT, 02Footprints:SW-SMD_SSSS810701, F.Cu at (147.7, 77.9)
- added U1: STM32F405RGT6, Package_QFP:LQFP-64_10x10mm_P0.5mm, F.Cu at (153.8, 95.5)
- added U2: AMS1117-3.3, Package_TO_SOT_SMD:SOT-223-3_TabPin2, F.Cu at (177.6, 113.2)
- added U3: USBLC6-2SC6, Package_TO_SOT_SMD:SOT-23-6, F.Cu at (166.5, 93.5)
- added U4: OPA350UA_2K5, 02Footprints:SOIC127P599X175-8N, F.Cu at (138.6, 104.5)
- added U5: OPA350UA_2K5, 02Footprints:SOIC127P599X175-8N, F.Cu at (140.2, 111.2)
- added Y1: 24MHz, Crystal:Crystal_SMD_3225-4Pin_3.2x2.5mm, F.Cu at (140.6, 90.8)
Routing:
- net +3.3V: track 0.00 -> 335.6 mm, vias 0 -> 13
- net /RESET: track 0.00 -> 95.0 mm
- net GND: track 0.00 -> 90.5 mm, vias 0 -> 43
- net /VBUS: track 0.00 -> 27.0 mm, vias 0 -> 2
- net /USART1_TX: track 0.00 -> 25.9 mm
- net /Encode_1: track 0.00 -> 25.9 mm, vias 0 -> 2
- net /CHL_Select: track 0.00 -> 24.7 mm
- net /LCD_MISO: track 0.00 -> 24.5 mm, vias 0 -> 1
- net /SWD_CLK: track 0.00 -> 24.3 mm
- net /LCD_CS: track 0.00 -> 24.1 mm
- net /USART1_RX: track 0.00 -> 23.8 mm
- net /LCD_RESET: track 0.00 -> 23.2 mm
- net /TIM2_1B: track 0.00 -> 22.7 mm
- net /SD_SCK: track 0.00 -> 22.7 mm
- net /SWD_IO: track 0.00 -> 22.5 mm
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- added copper zone on F.Cu, net +3.3V
- added copper zone on B.Cu, net GND
Other:
- board outline added: 68.1 x 55 mm
