File: Osciliscope PCB/Osciliscope PCB.kicad_sch (KiCad schematic)
At the start: 48 parts, among them J1 TYPE-C_16PIN_2MD__073_, J10 Conn_01x02_Pin, J11 Conn_01x04_Pin, J2 Conn_01x04_Pin, J3 Conn_01x09_Pin, J4 Conn_01x05_Pin, J5 Conn_01x05_Pin, J6 Conn_01x04_Pin, J7 Conn_01x03_Pin, J8 Conn_01x02_Pin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

Commit message: Edited Schematic
Parts:
- C1, C11, C14, C17, C18, C19, C20, C3, C4, C5, C6, C7: footprint Capacitor_SMD:C_0805_2012Metric -> (none); Part NO. C28233 -> (none)
- C10, C9: footprint Capacitor_SMD:C_0805_2012Metric -> (none); Part NO. C1797 -> (none)
- C12, C13, C2: footprint Capacitor_SMD:C_0805_2012Metric -> (none); Part NO. C15850 -> (none)
- C15, C16: footprint Capacitor_SMD:C_0805_2012Metric -> (none); Part NO. C377773 -> (none)
- C8: footprint Capacitor_SMD:C_0805_2012Metric -> (none); Part NO. C1779 -> (none)
- D2, D3: footprint LED_SMD:LED_0805_2012Metric -> (none); Part NO. C2295 -> (none)
- FB1: footprint Capacitor_SMD:C_0805_2012Metric -> (none); Part NO. C1017 -> (none)
- R1, R3: footprint Resistor_SMD:R_0805_2012Metric -> (none); Part NO. C17414 -> (none)
- R2, R4, R5, R6: footprint Resistor_SMD:R_0805_2012Metric -> (none); Part NO. C27834 -> (none)
- R24, R26: footprint Resistor_SMD:R_0805_2012Metric -> (none); Part NO. C17630 -> (none)
- SW1: Part NO. (none) -> C97433

Commit message: Edited schematic
Parts:
- C1, C10, C11, C14, C17, C18, C19, C20, C3, C4, C5, C6, C7, C9, R1, R2, R3, R4, R5, R6: footprint (none) -> Capacitor_SMD:C_0402_1005Metric
- C12, C13, C2, D2, D3, FB1: footprint (none) -> Capacitor_SMD:C_0805_2012Metric
- C15, C16, C8, R24, R26: footprint (none) -> Capacitor_SMD:C_0603_1608Metric
Changed lines of the file:
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@@
 			)
 		)
-		(property "Footprint" ""
+		(property "Footprint" "Capacitor_SMD:C_0402_1005Metric"
 			(at 132.588 175.26 90)
 			(effects
@@
 			)
 		)
-		(property "Footprint" ""
+		(property "Footprint" "Capacitor_SMD:C_0805_2012Metric"
 			(at 261.3152 86.36 0)
 			(effects
@@
 			)
 		)
-		(property "Footprint" ""
+		(property "Footprint" "Capacitor_SMD:C_0603_1608Metric"
 			(at 57.4548 120.65 0)
 			(effects
@@
 			)
 		)
-		(property "Footprint" ""
+		(property "Footprint" "Capacitor_SMD:C_0402_1005Metric"
 			(at 188.2648 36.83 0)
 			(effects
@@
 			)
 		)
-		(property "Footprint" ""
+		(property "Footprint" "Capacitor_SMD:C_0402_1005Metric"
 			(at 131.1148 55.88 0)
 			(effects
@@
 			)
 		)
-		(property "Footprint" ""
+		(property "Footprint" "Capacitor_SMD:C_0402_1005Metric"
 			(at 167.3352 36.83 0)
 			(effects
@@
 			)
 		)
-		(property "Footprint" ""
+		(property "Footprint" "Capacitor_SMD:C_0402_1005Metric"
 			(at 217.932 45.72 90)
 			(effects
@@
 			)
 		)
-		(property "Footprint" ""
+		(property "Footprint" "Capacitor_SMD:C_0402_1005Metric"
 			(at 50.4952 111.76 0)
 			(effects
@@
 			)
 		)
-		(property "Footprint" ""
+		(property "Footprint" "Capacitor_SMD:C_0402_1005Metric"
 			(at 41.148 158.75 90)
 			(effects
@@
 			)
 		)
-		(property "Footprint" ""
+		(property "Footprint" "Capacitor_SMD:C_0603_1608Metric"
 			(at 207.518 66.04 90)
 			(effects
@@
 			)
 		)
-		(property "Footprint" ""
+		(property "Footprint" "Capacitor_SMD:C_0402_1005Metric"
 			(at 46.6852 33.02 0)
 			(effects
@@
 			)
 		)
-		(property "Footprint" ""
+		(property "Footprint" "Capacitor_SMD:C_0805_2012Metric"
 			(at 23.8252 33.02 0)
 			(effects
@@
 			)
 		)
-		(property "Footprint" ""
+		(property "Footprint" "Capacitor_SMD:C_0402_1005Metric"
 			(at 164.7952 67.31 0)
 			(effects
@@
 			)
 		)
-		(property "Footprint" ""
+		(property "Footprint" "Capacitor_SMD:C_0603_1608Metric"
 			(at 64.4652 120.65 0)
 			(effects
@@
 			)
 		)
-		(property "Footprint" ""
+		(property "Footprint" "Capacitor_SMD:C_0402_1005Metric"
 			(at 69.5452 33.02 0)
 			(effects
@@
 			)
 		)
-		(property "Footprint" ""
+		(property "Footprint" "Capacitor_SMD:C_0402_1005Metric"
 			(at 80.9752 33.02 0)
 			(effects
@@
 			)
 		)
-		(property "Footprint" ""
+		(property "Footprint" "Capacitor_SMD:C_0402_1005Metric"
 			(at 272.542 45.72 90)
 			(effects
@@
 			)
 		)
-		(property "Footprint" ""
+		(property "Footprint" "Capacitor_SMD:C_0805_2012Metric"
 			(at 134.62 27.178 90)
 			(effects
@@
 			)
 		)
-		(property "Footprint" ""
+		(property "Footprint" "Capacitor_SMD:C_0402_1005Metric"
 			(at 132.842 175.26 90)
 			(effects
@@
 			)
 		)
-		(property "Footprint" ""
+		(property "Footprint" "Capacitor_SMD:C_0603_1608Metric"
 			(at 218.948 66.04 90)
 			(effects
@@
 			)
 		)
-		(property "Footprint" ""
+		(property "Footprint" "Capacitor_SMD:C_0402_1005Metric"
 			(at 37.7952 111.76 0)
 			(effects
@@
 			)
 		)
-		(property "Footprint" ""
+		(property "Footprint" "Capacitor_SMD:C_0402_1005Metric"
 			(at 69.85 166.878 90)
 			(effects
@@
 			)
 		)
-		(property "Footprint" ""
+		(property "Footprint" "Capacitor_SMD:C_0402_1005Metric"
 			(at 112.7252 33.02 0)
 			(effects
@@
 			)
 		)
-		(property "Footprint" ""
+		(property "Footprint" "Capacitor_SMD:C_0402_1005Metric"
 			(at 26.3652 111.76 0)
 			(effects
@@
 			)
 		)
-		(property "Footprint" ""
+		(property "Footprint" "Capacitor_SMD:C_0805_2012Metric"
 			(at 217.17 74.93 0)
 			(effects
@@
 			)
 		)
-		(property "Footprint" ""
+		(property "Footprint" "Capacitor_SMD:C_0603_1608Metric"
 			(at 123.4948 33.02 0)
 			(effects
@@
 			)
 		)
-		(property "Footprint" ""
+		(property "Footprint" "Capacitor_SMD:C_0402_1005Metric"
 			(at 58.1152 33.02 0)
 			(effects
@@
 			)
 		)
-		(property "Footprint" ""
+		(property "Footprint" "Capacitor_SMD:C_0805_2012Metric"
 			(at 237.1852 86.36 0)
 			(effects
@@
 			)
 		)
-		(property "Footprint" ""
+		(property "Footprint" "Capacitor_SMD:C_0805_2012Metric"
 			(at 205.74 74.93 0)
 			(effects
@@
 			)
 		)
-		(property "Footprint" ""
+		(property "Footprint" "Capacitor_SMD:C_0402_1005Metric"
 			(at 35.2552 33.02 0)
 			(effects
@@
 			)
 		)
-		(property "Footprint" ""
+		(property "Footprint" "Capacitor_SMD:C_0402_1005Metric"
 			(at 31.4452 175.26 0)
 			(effects

Commit message: Finished PCB
Parts:
- added C28: 100n, Capacitor_SMD:C_0402_1005Metric, symbol Device:C
Connections:
- net GND: now also C28.2
- net Scale_Axis: now also C28.1
- net 5V_LED: now reaches D2.2 (A), R24.2
- net 3V_LED: now reaches D3.2 (A), R26.2
Other:
- moved on the sheet: R24, R26
Changed lines of the file:
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@@
 	(wire
 		(pts
-			(xy 217.17 59.69) (xy 217.17 62.23)
+			(xy 217.17 59.69) (xy 217.17 60.96)
 		)
 		(stroke
@@
 	(wire
 		(pts
-			(xy 205.74 69.85) (xy 205.74 71.12)
+			(xy 205.74 68.58) (xy 205.74 71.12)
 		)
 		(stroke
@@
 	(wire
 		(pts
-			(xy 113.03 96.52) (xy 110.49 96.52)
+			(xy 110.49 96.52) (xy 127 96.52)
 		)
 		(stroke
@@
 	(wire
 		(pts
-			(xy 205.74 59.69) (xy 205.74 62.23)
+			(xy 205.74 59.69) (xy 205.74 60.96)
 		)
 		(stroke
@@
 	(wire
 		(pts
+			(xy 127 104.14) (xy 127 105.41)
+		)
+		(stroke
+			(width 0)
+			(type default)
+		)
+	)
+	(wire
+		(pts
 			(xy 168.91 90.17) (xy 152.4 90.17)
 		)
@@
 	(wire
 		(pts
-			(xy 217.17 69.85) (xy 217.17 71.12)
+			(xy 217.17 68.58) (xy 217.17 71.12)
 		)
 		(stroke
@@
 		)
 	)
+	(label "3V_LED"
+		(at 217.17 69.85 0)
+		(effects
+			(font
+				(size 1.27 1.27)
+			)
+			(justify left bottom)
+		)
+	)
 	(label "HSE_IN"
 		(at 172.72 26.67 180)
@@
 		)
 	)
+	(label "5V_LED"
+		(at 205.74 69.85 0)
+		(effects
+			(font
+				(size 1.27 1.27)
+			)
+			(justify left bottom)
+		)
+	)
 	(label "Encode_2"
 		(at 191.77 120.65 0)
@@
 	(symbol
 		(lib_id "Device:R")
-		(at 205.74 66.04 0)
+		(at 205.74 64.77 0)
 		(mirror y)
 		(unit 1)
@@
 		(fields_autoplaced yes)
 		(property "Reference" "R24"
-			(at 208.28 64.7699 0)
+			(at 208.28 63.4999 0)
 			(effects
 				(font
@@
 		)
 		(property "Value" "330"
-			(at 208.28 67.3099 0)
+			(at 208.28 66.0399 0)
 			(effects
 				(font
@@
 		)
 		(property "Footprint" "Capacitor_SMD:C_0603_1608Metric"
-			(at 207.518 66.04 90)
+			(at 207.518 64.77 90)
 			(effects
 				(font
@@
 		)
 		(property "Datasheet" ""
-			(at 205.74 66.04 0)
+			(at 205.74 64.77 0)
 			(effects
 				(font
@@
 		)
 		(property "Description" ""
-			(at 205.74 66.04 0)
+			(at 205.74 64.77 0)
 			(effects
 				(font
@@
 		)
 		(property "Part NO." ""
-			(at 205.74 66.04 0)
+			(at 205.74 64.77 0)
 			(effects
 				(font
@@
 	)
 	(symbol
+		(lib_id "Device:C")
+		(at 127 100.33 0)
+		(mirror y)
+		(unit 1)
+		(exclude_from_sim no)
+		(in_bom yes)
+		(on_board yes)
+		(dnp no)
+		(property "Reference" "C28"
+			(at 130.81 99.0599 0)
+			(effects
+				(font
+					(size 1.27 1.27)
+				)
+				(justify right)
+			)
+		)
+		(property "Value" "100n"
+			(at 130.81 101.5999 0)
+			(effects
+				(font
+					(size 1.27 1.27)
+				)
+				(justify right)
+			)
+		)
+		(property "Footprint" "Capacitor_SMD:C_0402_1005Metric"
+			(at 126.0348 104.14 0)
+			(effects
+				(font
+					(size 1.27 1.27)
+				)
+				(hide yes)
+			)
+		)
+		(property "Datasheet" ""
+			(at 127 100.33 0)
+			(effects
+				(font
+					(size 1.27 1.27)
+				)
+				(hide yes)
+			)
+		)
+		(property "Description" ""
+			(at 127 100.33 0)
+			(effects
+				(font
+					(size 1.27 1.27)
+				)
+				(hide yes)
+			)
+		)
+		(property "Part NO." ""
+			(at 127 100.33 0)
+			(effects
+				(font
+					(size 1.27 1.27)
+				)
+				(hide yes)
+			)
+		)
+		(pin "1"
+		)
+		(pin "2"
+		)
+		(instances
+			(project "Osciliscope PCB"
+				(path "/dbd44bf2-721f-49a6-94a9-d8437df40c50"
+					(reference "C28")
+					(unit 1)
+				)
+			)
+		)
+	)
+	(symbol
 		(lib_id "Device:R")
 		(at 274.32 45.72 0)
@@
 	(symbol
 		(lib_id "Device:R")
-		(at 217.17 66.04 0)
+		(at 217.17 64.77 0)
 		(mirror y)
 		(unit 1)
@@
 		(fields_autoplaced yes)
 		(property "Reference" "R26"
-			(at 219.71 64.7699 0)
+			(at 219.71 63.4999 0)
 			(effects
 				(font
@@
 		)
 		(property "Value" "330"
-			(at 219.71 67.3099 0)
+			(at 219.71 66.0399 0)
 			(effects
 				(font
@@
 		)
 		(property "Footprint" "Capacitor_SMD:C_0603_1608Metric"
-			(at 218.948 66.04 90)
+			(at 218.948 64.77 90)
 			(effects
 				(font
@@
 		)
 		(property "Datasheet" ""
-			(at 217.17 66.04 0)
+			(at 217.17 64.77 0)
 			(effects
 				(font
@@
 		)
 		(property "Description" ""
-			(at 217.17 66.04 0)
+			(at 217.17 64.77 0)
 			(effects
 				(font
@@
 		)
 		(property "Part NO." ""
-			(at 217.17 66.04 0)
+			(at 217.17 64.77 0)
 			(effects
 				(font
@@
 					(unit 1)
 				)
+			)
+		)
+	)
+	(symbol
+		(lib_id "power:GND")
+		(at 127 105.41 0)
+		(unit 1)
+		(exclude_from_sim no)
+		(in_bom yes)
+		(on_board yes)
+		(dnp no)
+		(fields_autoplaced yes)
+		(property "Reference" "#PWR019"
+			(at 127 111.76 0)
+			(effects
+				(font
+					(size 1.27 1.27)
+				)
+				(hide yes)
+			)
+		)
+		(property "Value" "GND"
+			(at 127 110.49 0)
+			(effects
+				(font
+					(size 1.27 1.27)
+				)
+			)
+		)
+		(property "Footprint" ""
+			(at 127 105.41 0)
+			(effects
+				(font
+					(size 1.27 1.27)
+				)
+				(hide yes)
+			)
+		)
+		(property "Datasheet" ""
+			(at 127 105.41 0)
+			(effects
+				(font
+					(size 1.27 1.27)
+				)
+				(hide yes)
+			)
+		)
+		(property "Description" "Power symbol creates a global label with name \"GND\" , ground"
+			(at 127 105.41 0)
+			(effects
+				(font
+					(size 1.27 1.27)
+				)
+				(hide yes)
+			)
+		)
+		(pin "1"
+		)
+		(instances
+			(project "Osciliscope PCB"
+				(path "/dbd44bf2-721f-49a6-94a9-d8437df40c50"
+					(reference "#PWR019")
+					(unit 1)
+				)
